File: Design/M3DUBoard_V1.kicad_sch (KiCad schematic)
At the start: 398 parts, among them IC1 STM32F103RBT6, IC2 STM32F107VCT6, IC3 MLX91209LVA-CAA-000-SP, IC4 MLX91209LVA-CAA-000-SP, J1 Conn_01x30_Male, Q181 WVS, Q182 WVS, Q183 WVS, Q211 3N0408, Q212 3N0408, Q213 3N0408, Q301 WSB, Q302 WSB, Q303 WSB, Q311 WVS, Q312 WVS, Q313 WVS, Q321 WSB, Q322 WSB, Q323 WSB, Q41 45P4LLF6, Q42 45P4LLF6, Q43 45P4LLF6, Q51 SG NMOS D, Q52 SG NMOS D, Q53 SG NMOS D, Q981 45P4LLF6, Q982 45P4LLF6, Q983 45P4LLF6, Q991 3N0408, Q992 3N0408, Q993 3N0408, U10 TPS565208, U11 ACPL-C87A, U291 STGAP1AS, U292 STGAP1AS, U293 STGAP1AS, U301 STGAP1AS, U302 STGAP1AS, U303 STGAP1AS, U7 SN65HVD230, U8 SN65HVD230, U9 TPS565208

Commit message: Update Gate Driver schematic
Parts:
- added D2, D3, D421, D491, D492, D493: VN17, Diode_SMD:D_SMA, symbol Device:D
- added ST1, ST3, ST4: Thermistor, Connector_PinHeader_2.54mm:PinHeader_1x02_P2.54mm_Vertical, symbol Device:Thermistor
- R1291, R1292, R1293, R1561, R1562, R1563: value 189? -> 189
- R191, R192, R193, R196, R197, R227, R267, R268, R301: value 1004 -> 1M
Connections:
- net HV-: now also R267.2, R268.2, R301.2
- net VL_LS: now reaches C2571.1, C294.1, D53.2 (A), U301.23 (VL)
- net VL_LS: now also C2572.1, C2573.1, C2581.1, C2582.1, C2583.1, C2591.2, C2592.2, C2593.2, C301.1, C304.1, D61.2 (A), D62.2 (A), Q211.3 (S), Q212.3 (S), Q213.3 (S), Q321.2 (S), Q322.2 (S), Q323.2 (S), R1721.2, R1722.2, R1723.2, R1761.1, R1762.1, R1763.1, U301.14 (VL), U302.14 (VL), U302.23 (VL), U303.14 (VL), U303.23 (VL)
- net μC_MOSI: now reaches R1533.2
- net μC_MOSI: no longer R1463.2
- net at D1061.1 (K), R4061.2, R5061.2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: now also D1041.1 (K), D1051.1 (K), D1071.1 (K), R4041.2, R4051.2, R4071.2, R5041.2, R5051.2, R5071.2, R6041.2, R6051.2, R6061.2, R6071.2, TR1.1 (Source1), TR1.2 (Gate1), TR1.3 (Source2), TR1.4 (Gate2), TR1.5 (Source3), TR1.7 (Source4), TR1.8 (Gate4)
- net SDI_A: now reaches R1531.2
- net SDI_A: now also U292.2 (SDO); no longer R1461.2
- net GND_ISO_C: now reaches C2342.2, C2352.2, C2362.2, C2412.2, C2422.2, C2432.1, C2562.1, C2692.1, D412.2 (A), R6002.1, R6012.1, R6022.1, R6032.1, TP1412.1, U292.13 (GNDISO), U292.24 (ASC)
- net VL_HS_C: now reaches C2422.1, C2432.2, Q302.2 (S), Q52.1 (G), Q992.3 (S), U292.14 (VL)
- net VL_HS_C: now also C2412.1, R1652.2, R1662.1, U292.23 (VL)
- net VH_LS_C: now reaches C2492.1, C2502.1, D77.1 (K), Q312.2 (S), Q42.3 (S), U302.17 (VH)
- net VH_LS_C: now also R1692.2, R1702.1, D492.1 (K)
- net GND_ISO_B: now reaches C2343.2, C2353.2, C2363.2, C2413.2, C2423.2, C2433.1, C2563.1, C2693.1, D413.2 (A), R6003.1, R6013.1, R6023.1, R6033.1, TP1413.1, U293.13 (GNDISO), U293.24 (ASC)
- net VL_HS_B: now reaches C2421.1, C2431.2, Q301.2 (S), Q51.1 (G), Q991.3 (S), U291.14 (VL)
- net VL_HS_B: now also C2411.1, C2413.1, C2423.1, C2433.2, Q303.2 (S), Q53.1 (G), Q993.3 (S), R1651.2, R1661.1, R1663.1, R1853.2, U291.23 (VL), U293.14 (VL), U293.23 (VL)
- net VH_HS_B: now reaches C2353.1, C2363.1, Q183.2 (S), Q983.3 (S), U293.17 (VH)
- net VH_HS_B: now also R1583.2, R1633.1
- net μC_PWM_B_P: now reaches R1413.2
- net μC_CK: now reaches R1291.2
- net μC_CK: now also R1292.2, R1293.2, R1561.2, R1562.2, R1563.2; no longer R1471.2
- net VH_HS_C: now reaches R1582.2, R1632.1
- net VH_HS_C: now also C2352.1, C2362.1, Q182.2 (S), Q982.3 (S), U292.17 (VH)
- net ASC_L: now reaches R3212.1, TP1452.1, U302.24 (ASC)
- net ASC_L: now also R3211.1, R3213.1, TP1451.1, TP1453.1, U301.24 (ASC), U303.24 (ASC)
- net at R1481.2: now also D483.2 (A); no longer D481.2 (A)
- net GND_ISO_A: now reaches C2341.2, C2351.2, C2361.2, C2411.2, C2421.2, C2431.1, C2561.1, C2691.1, D411.2 (A), R6001.1, R6011.1, R6021.1, R6031.1, TP1411.1, U291.13 (GNDISO), U291.24 (ASC)
- net +3.3V: now reaches C2371.2, C2401.2, C2521.2, C2701.2, U291.6 (VREG), U301.6 (VREG)
- net +3.3V: now also C2372.2, C2373.2, C2402.2, C2403.2, C2522.2, C2523.2, C2702.2, C2703.2, U291.7 (VDD), U292.6 (VREG), U292.7 (VDD), U293.6 (VREG), U293.7 (VDD), U302.6 (VREG), U303.6 (VREG)
- net μC_DIAG: now reaches TP1362.1, U292.10 (DIAG1), U302.10 (DIAG1)
- net μC_DIAG: now also TP1361.1, TP1363.1, U291.10 (DIAG1), U293.10 (DIAG1), U301.10 (DIAG1), U303.10 (DIAG1)
- net μC_~CS: now reaches R1473.2
- net μC_~CS: now also R1461.2, R1462.2, R1463.2, R1471.2, R1472.2; no longer R1293.2
- net VH_HS_A: now reaches C2351.1, C2361.1, Q181.2 (S), Q981.3 (S), U291.17 (VH)
- net VH_HS_A: now also R1581.2, R1631.1
- net VH_LS_B: now reaches R1693.2, R1703.1
- net VH_LS_B: now also C2491.1, C2493.1, C2501.1, C2503.1, D74.1 (K), D78.1 (K), Q311.2 (S), Q313.2 (S), Q41.3 (S), Q43.3 (S), R1691.2, R1701.1, U301.17 (VH), U303.17 (VH), D491.1 (K), D493.1 (K)
- net at D481.1 (K): now also U293.16 (SENSE); no longer U291.16 (SENSE)
- net at D483.1 (K): now also U291.16 (SENSE); no longer U293.16 (SENSE)
- net SDI_C: now reaches U293.2 (SDO)
- net SDI_C: now also R1532.2
- net μC_PWM_C_N: now reaches R1592.2
- net μC_PWM_A_N: now reaches R1591.2
- net at R1483.2: now also D481.2 (A); no longer D483.2 (A)
- net μC_MISO: now reaches U291.2 (SDO)
- net μC_PWM_C_P: now reaches R1412.2
- net μC_PWM_B_N: now reaches R1593.2
- net μC_~SD: now reaches R1452.2, TP58.1
- net μC_~SD: now also R1451.2, R1453.2
- net μC_PWM_A_P: now reaches R1411.2
- net at R1333.2: now also D3.2 (A)
- net at R1332.2: now also D2.2 (A)
- net at R1331.2: now also D421.2 (A)
- new net DSAT_A: D421.1 (K)
- new net DSAT_B: D3.1 (K)
- new net DSAT_C: D2.1 (K)
- new net VH_LS: D491.2 (A), D492.2 (A), D493.2 (A)
Other:
- note added: "Gate Driver, Phase A"
- note added: "Gate Driver, Phase B"
- note added: "Gate Driver, Phase C"
- note added: "Legend: ------------------------------------------- VH_HS_A - Positive power supply for HV section, High Side, Phase A VL_HS_A - Negative power supply for HV section, High Side, Phase A VH_LS_A - Positive power supply for HV section, Low Side, Phase C VH_HS_B - Positive power supply for HV section, High Side, Phase B VL_HS_B - Negative power supply for HV section, High Side, Phase B VH_LS_B - Pos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"
- company: (none) -> EVBMW.COM, OPENINVERTER.ORG
- title: (none) -> M3DU Logic Board
- moved on the sheet: C2001, C2002, C2003, C2341, C2342, C2343, C2351, C2352, C2353, C2361, C2362, C2363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
